File: KiCad/Apple_II_RAM-ROM128_GAL.kicad_pcb (KiCad board)
At the start: 4 copper layers, 114.9 x 79 mm, 30 parts, among them J1 Apple ][ Bus, U1 HM628128, U2 29F010, U3 GAL22V10, U4 GAL22V10

Commit message: design update
Parts:
- SATURN: moved to B.Cu
- moved OSHW1 110.9 mm to (205.1, 71.8)
- moved REF** 110.9 mm to (205.1, 71.8)
- moved SATURN 33.6 mm to (191.8, 99.1), turned to 180 degrees
Other:
- board text added: "GAL RAM"
- board text added: "GAL ROM"
